File: dev/FalloutProject.kicad_sch (KiCad schematic)
At the start: 60 parts, among them Q1 2N3904, Q2 2N3904, Q3 2N3904, Q4 2N3904, SW1 SW_Push, SW2 SW_Push, SW3 SW_Push

Commit message: commit before merge with commit: Add demo logic diagram
Parts:
- added LA2: Lamp, symbol Device:Lamp
- added Q5: 2N3904, Package_TO_SOT_THT:TO-92_Inline, symbol Transistor_BJT:2N3904
- added Q6: KPS-3227, OptoDevice:Kingbright_KPS-3227, symbol Sensor_Optical:KPS-3227
- added R10, R6: R, symbol Device:R
Connections:
- net GND: now also LA2.1 (-), Q5.1 (E), Q6.2, Q6.4
- net VCC: now also R10.2, R6.2
- new net: Q5.2 (B), Q6.1, Q6.3, R6.1
- new net: LA2.2 (+), Q5.3 (C), R10.1
