File: components/redstone-repeater/redstone-repeater.kicad_sch (KiCad schematic)
At the start: 21 parts, among them Q1 2N3904, Q13 Q_NMOS_DGS, Q14 Q_NMOS_DGS, Q15 Q_NMOS_DGS, Q16 Q_NMOS_DGS, Q2 2N3904, Q3 2N3904, Q4 2N3904, SW1 SW_Push, SW2 SW_Push

Commit message: commit before merge with commit: Add demo logic diagram
Parts:
- added LA2: Lamp, symbol Device:Lamp
- added Q5, Q6: 2N3904, Package_TO_SOT_THT:TO-92_Inline, symbol Transistor_BJT:2N3904
- added Q7, Q8: KPS-3227, OptoDevice:Kingbright_KPS-3227, symbol Sensor_Optical:KPS-3227
- added R1: R, symbol Device:R
Connections:
- net GND: now also LA2.1 (-), LA2.2 (+), R1.2
- net VCC: now also Q5.3 (C), Q7.2, Q7.4, Q8.2, Q8.4
- new net: Q6.1 (E), R1.1
- new net: Q5.2 (B), Q8.1, Q8.3
- new net: Q6.2 (B), Q7.1, Q7.3
- new net: Q5.1 (E), Q6.3 (C)

Commit message: Update component schematics
Parts:
- added D1: LED, symbol Device:LED
- added Q16, Q18: PT928-6C-F, symbol Device:Q_Photo_NPN
- added Q17, Q19: S9014, PCM_JLCPCB:Q_SOT-23, symbol PCM_JLCPCB-Transistors:NPN,S9014
- added R15, R17: 75k, symbol Device:R
- added R16: 100, symbol Device:R
- renumbered LA2 to LA1, LA1 to LA2, Q5 to Q10, Q6 to Q11, Q3 to Q12, Q1 to Q13, Q2 to Q14, Q4 to Q15, Q13 to Q4, Q15 to Q5, Q14 to Q6, Q16 to Q7, Q7 to Q9, R47 to R10, R43 to R11, R7 to R12, R48 to R13, R49 to R14, R44 to R4, R42 to R5, R46 to R7, R45 to R8, R1 to R9
Connections:
- net GND: now also Q19.2 (E), R15.2, R17.2
- net VCC: now also Q16.1 (C), Q18.1 (C), R16.1
- new net: Q16.2 (E), Q17.1 (B), R15.1
- new net: D1.2 (A), R16.2
- new net: Q18.2 (E), Q19.1 (B), R17.1
- new net: D1.1 (K), Q17.3 (C)
- new net: Q17.2 (E), Q19.3 (C)
Other:
- moved on the sheet: LA1, Q10, Q11, Q8, Q9, R9
