File: components/redstone-torch/redstone-torch.kicad_sch (KiCad schematic)
At the start: 8 parts, among them Q12 Q_NMOS_DGS, Q4 2N3904, SW3 SW_Push

Commit message: commit before merge with commit: Add demo logic diagram
Parts:
- removed SW3: SW_Push, symbol Switch:SW_Push
- added Q1: Q_Photo_NPN, symbol Device:Q_Photo_NPN
- R8: value R -> 15k
- R9: value R -> 100
Connections:
- net VCC: now also Q1.1 (C)
- net at R8.1: now also Q1.2 (E)
Changed lines of the file:
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@@
-	)
-	(symbol
-		(lib_id "Switch:SW_Push")
-		(at 60.96 78.74 0)
-		(unit 1)
-		(body_style 1)
-		(exclude_from_sim no)
-		(in_bom yes)
-		(on_board yes)
-		(in_pos_files yes)
-		(dnp no)
-		(fields_autoplaced yes)
-		(property "Reference" "SW3"
-			(at 60.96 71.12 0)
-			(show_name no)
-			(do_not_autoplace no)
-			(effects
-				(font
-					(size 1.27 1.27)
-				)
-			)
-		)
-		(property "Value" "SW_Push"
-			(at 60.96 73.66 0)
-			(show_name no)
-			(do_not_autoplace no)
-			(effects
-				(font
-					(size 1.27 1.27)
-				)
-			)
-		)
-		(property "Footprint" ""
-			(at 60.96 73.66 0)
-			(hide yes)
-			(show_name no)
-			(do_not_autoplace no)
-			(effects
-				(font
-					(size 1.27 1.27)
-				)
-			)
-		)
-		(property "Datasheet" ""
-			(at 60.96 73.66 0)
-			(hide yes)
-			(show_name no)
-			(do_not_autoplace no)
-			(effects
-				(font
-					(size 1.27 1.27)
-				)
-			)
-		)
-		(property "Description" "Push button switch, generic, two pins"
-			(at 60.96 78.74 0)
-			(hide yes)
-			(show_name no)
-			(do_not_autoplace no)
-			(effects
-				(font
-					(size 1.27 1.27)
-				)
-			)
-		)
-		(pin "2"
-		)
-		(pin "1"
-		)
-		(instances
-			(project "redstone-torch"
-				(path "/5d24c42e-ea6a-418f-a288-e53a0e2e8e34"
-					(reference "SW3")
-					(unit 1)
-				)
-			)
-		)
 	)
 	(symbol
@@
 			)
 		)
-		(property "Value" "R"
+		(property "Value" "100"
 			(at 91.44 83.8199 0)
 			(show_name no)
@@
 			)
 		)
-		(property "Value" "R"
+		(property "Value" "15k"
 			(at 73.66 74.93 90)
 			(show_name no)
@@
 					(unit 1)
 				)
+			)
+		)
+	)
+	(symbol
+		(lib_id "Device:Q_Photo_NPN")
+		(at 60.96 81.28 90)
+		(unit 1)
+		(body_style 1)
+		(exclude_from_sim no)
+		(in_bom yes)
+		(on_board yes)
+		(in_pos_files yes)
+		(dnp no)
+		(fields_autoplaced yes)
+		(property "Reference" "Q1"
+			(at 60.2107 72.39 90)
+			(show_name no)
+			(do_not_autoplace no)
+			(effects
+				(font
+					(size 1.27 1.27)
+				)
+			)
+		)
+		(property "Value" "Q_Photo_NPN"
+			(at 60.2107 74.93 90)
+			(show_name no)
+			(do_not_autoplace no)
+			(effects
+				(font
+					(size 1.27 1.27)
+				)
+			)
+		)
+		(property "Footprint" ""
+			(at 58.42 76.2 0)
+			(hide yes)
+			(show_name no)
+			(do_not_autoplace no)
+			(effects
+				(font
+					(size 1.27 1.27)
+				)
+			)
+		)
+		(property "Datasheet" ""
+			(at 60.96 81.28 0)
+			(hide yes)
+			(show_name no)
+			(do_not_autoplace no)
+			(effects
+				(font
+					(size 1.27 1.27)
+				)
+			)
+		)
+		(property "Description" "NPN phototransistor, collector/emitter"
+			(at 60.96 81.28 0)
+			(hide yes)
+			(show_name no)
+			(do_not_autoplace no)
+			(effects
+				(font
+					(size 1.27 1.27)
+				)
+			)
+		)
+		(pin "2"
+		)
+		(pin "1"
+		)
+		(instances
+			(project "redstone-torch"
+				(path "/5d24c42e-ea6a-418f-a288-e53a0e2e8e34"
+					(reference "Q1")
+					(unit 1)
+				)

Commit message: Update component schematics
Parts:
- added D2: LED, symbol Device:LED
- added Q23: PT928-6C-F, symbol Device:Q_Photo_NPN
- added Q24: S9014, PCM_JLCPCB:Q_SOT-23, symbol PCM_JLCPCB-Transistors:NPN,S9014
- added R22: 15k, symbol Device:R
- added R23: 100, symbol Device:R
- renumbered LA1 to LA3, Q1 to Q20, Q12 to Q21, Q4 to Q22, R41 to R18, R8 to R19, R43 to R20, R9 to R21
Connections:
- net GND: now also Q23.2 (E), Q24.2 (E)
- net VCC: now also R22.2, R23.2
- new net: Q23.1 (C), Q24.1 (B), R22.1
- new net: D2.1 (K), Q24.3 (C)
- new net: D2.2 (A), R23.1
